File: Resources/Electronics/Kaffettino/Kaffettino.kicad_pcb (KiCad board)
At the start: 2 copper layers, 43 parts, among them J1 PPTC101LFBN-RC, J2 USB_C_Receptacle_PowerOnly_6P, M1 RFID-RC522, SW1 SW_Push, U2 DFR0299

Commit message: Added expansion pins and changed power method in electrical schema
Parts:
- removed R12: 5.1k, Resistor_THT:R_Axial_DIN0207_L6.3mm_D2.5mm_P10.16mm_Horizontal
- removed R23: 10k, Resistor_THT:R_Axial_DIN0207_L6.3mm_D2.5mm_P10.16mm_Horizontal
- removed SW1: SW_Push, OSTVN02A150:CONN_OSTVN02A150_OST
- added C6: 100nF, Capacitor_THT:C_Disc_D3.0mm_W1.6mm_P2.50mm, F.Cu at (247.1, 66.0)
- added R25: 1k, Resistor_THT:R_Axial_DIN0207_L6.3mm_D2.5mm_P10.16mm_Horizontal, F.Cu at (214.0, 76.1)
- added U3: DFR0299, DFR0299:MODULE_DFR0299, F.Cu at (58.5, 45.0)
- C10: value 100nF -> 4.7uF; footprint Capacitor_THT:C_Disc_D3.0mm_W1.6mm_P2.50mm -> Capacitor_THT:CP_Radial_D6.3mm_P2.50mm
- J2: value USB_C_Receptacle_PowerOnly_6P -> OSTVN02A150; footprint Connector_USB:USB_C_Receptacle_GCT_USB4125-xx-x_6P_TopMnt_Horizontal -> OSTVN02A150:CONN_OSTVN02A150_OST
- R10, R20, R21: value 1k -> 10k
- R13: value 5.1k -> 1k
- R18, R6: value 10k -> 1k
- U1: value ~ -> PCF8574AN; footprint ESP32-38Pin:ESP32_38pin -> PCF8574AN:N16
- U2: value DFR0299 -> ESP32-38Pin-Wroom; footprint DFR0299:MODULE_DFR0299 -> ESP32-38Pin:ESP32_38pin
- moved J1 222.7 mm to (277.6, 18.8), turned to -90 degrees
- moved C1 203.7 mm to (266.1, 66.0), turned to -90 degrees
- moved C2 194.8 mm to (256.6, 66.0), turned to -90 degrees
- moved C7 178.2 mm to (237.6, 66.0), turned to -90 degrees
- moved R8 165.7 mm to (270.6, 76.1), turned to 90 degrees
- moved R4 161.5 mm to (266.1, 56.3), turned to 90 degrees
- moved R5 152.4 mm to (256.6, 56.3), turned to 90 degrees
- moved C3 150.4 mm to (210.5, 66.0), turned to -90 degrees
- moved C4 144.7 mm to (203.8, 66.0), turned to -90 degrees
- moved R9 143.7 mm to (261.1, 76.1), turned to 90 degrees
- moved C8 140.4 mm to (197.1, 66.0), turned to -90 degrees
- moved C9 135.3 mm to (190.5, 66.0), turned to -90 degrees
- moved R15 131.1 mm to (247.1, 56.3), turned to 90 degrees
- moved R16 122.8 mm to (237.6, 56.3), turned to 90 degrees
- moved R19 120.2 mm to (251.6, 76.1), turned to 90 degrees
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Connections:
- Brd1 pad 3: /OLED_SCL -> /GEN_SCL
- Brd1 pad 4: /OLED_SDA -> /GEN_SDA
- C1 pad 1: /KP_C3 -> /KP_R4
- C10 pad 1: /KP_R1 -> +5V
- C2 pad 1: /KP_C2 -> /KP_R3
- C4 pad 1: /KP_C1 -> /KP_C3
- C7 pad 1: /KP_R4 -> /KP_R1
- C8 pad 1: /KP_R3 -> /KP_C2
- C9 pad 1: /KP_R2 -> /KP_C1
- LS1 pad 1: Net-(U2-SPK1) -> Net-(U3-SPK1)
- LS1 pad 2: Net-(U2-SPK2) -> Net-(U3-SPK2)
- R10 pad 1: /KP_C1 -> +3.3V
- R10 pad 2: Net-(J1-Pad2) -> /KP_C4
- R11 pad 2: /KP_C1 -> /KP_C3
- R13 pad 1: Net-(J2-CC1) -> +3.3V
- R13 pad 2: GNDREF -> /GEN_SDA
- R14 pad 2: /OLED_SDA -> /GEN_SCL
- R15 pad 1: +3.3V -> /KP_R2
- R15 pad 2: /OLED_SCL -> Net-(J1-Pad7)
- R16 pad 1: /KP_R4 -> /KP_R1
- R16 pad 2: Net-(J1-Pad9) -> Net-(J1-Pad6)
- R17 pad 1: /KP_R3 -> /KP_C2
- R17 pad 2: Net-(J1-Pad8) -> Net-(J1-Pad3)
- R18 pad 1: +3.3V -> /KP_C1
- R18 pad 2: /KP_R4 -> Net-(J1-Pad2)
- R19 pad 2: /KP_R3 -> /KP_R2
- R20 pad 1: /KP_R2 -> +3.3V
- R20 pad 2: Net-(J1-Pad7) -> /KP_R1
- R21 pad 1: /KP_R1 -> +3.3V
- R21 pad 2: Net-(J1-Pad6) -> /KP_C2
- R22 pad 2: /KP_R2 -> /KP_C1
- R4 pad 1: /KP_C3 -> /KP_R4
- R4 pad 2: Net-(J1-Pad4) -> Net-(J1-Pad9)
- R5 pad 1: /KP_C4 -> /KP_R3
- R5 pad 2: Net-(J1-Pad5) -> Net-(J1-Pad8)
- R6 pad 1: +3.3V -> /KP_C4
- R6 pad 2: /KP_C3 -> Net-(J1-Pad5)
- R7 pad 1: /KP_C2 -> /KP_C3
- R7 pad 2: Net-(J1-Pad3) -> Net-(J1-Pad4)
- R8 pad 2: /KP_C4 -> /KP_R4
- R9 pad 2: /KP_C2 -> /KP_R3
- U1 pad 1: +5V -> GNDREF
- U1 pad 10: /GREEN -> /KP_C2
- U1 pad 11: unconnected-(U1-GPIO25-Pad11) -> /KP_C3
- U1 pad 12: /MICRO_SD_RX -> /KP_C4
- U1 pad 13: /MICRO_SD_TX -> Net-(U1-*INT)
- U1 pad 14: unconnected-(U1-GPIO35-Pad14) -> /GEN_SCL
- U1 pad 15: /RFID_RST -> /GEN_SDA
- U1 pad 16: unconnected-(U1-GPIO39-Pad16) -> +3.3V
- U1 pad 2: unconnected-(U1-GPIO11-Pad2) -> GNDREF
- U1 pad 3: unconnected-(U1-GPIO10-Pad3) -> GNDREF
- U1 pad 4: unconnected-(U1-GPIO9-Pad4) -> /KP_R1
- U1 pad 5: unconnected-(U1-GPIO13-Pad5) -> /KP_R2
- U1 pad 6: GNDREF -> /KP_R3
- U1 pad 7: unconnected-(U1-GPIO12-Pad7) -> /KP_R4
- U1 pad 8: /RED -> GNDREF
- U1 pad 9: /YELLOW -> /KP_C1
- U2 pad 1: +3.3V -> +5V
- U2 pad 10: GNDREF -> /GREEN
- U2 pad 12: unconnected-(U2-ADKEY1-Pad12) -> /MICRO_SD_RX
- U2 pad 13: unconnected-(U2-ADKEY2-Pad13) -> /MICRO_SD_TX
- U2 pad 15: unconnected-(U2-USB--Pad15) -> /RFID_RST
- U2 pad 2: /MICRO_SD_RX -> unconnected-(U2-GPIO11-Pad2)
- U2 pad 3: /MICRO_SD_TX -> unconnected-(U2-GPIO10-Pad3)
- U2 pad 6: Net-(U2-SPK1) -> GNDREF
- U2 pad 7: GNDREF -> unconnected-(U2-GPIO12-Pad7)
- U2 pad 8: Net-(U2-SPK2) -> /RED
- U2 pad 9: unconnected-(U2-IO1-Pad9) -> /YELLOW
Routing:
- net GNDREF: track 0.00 -> 276.2 mm
- net +3.3V: track 0.00 -> 125.8 mm
- net Net-(J1-Pad2): track 0.00 -> 95.5 mm
- net Net-(J1-Pad3): track 0.00 -> 86.9 mm
- net Net-(J1-Pad4): track 0.00 -> 78.4 mm
- net /RED: track 0.00 -> 77.7 mm
- net /YELLOW: track 0.00 -> 75.6 mm
- net /GREEN: track 0.00 -> 73.6 mm
- net Net-(J1-Pad5): track 0.00 -> 69.8 mm
- net /KP_R4: track 0.00 -> 55.7 mm
- net /KP_C1: track 0.00 -> 47.6 mm
- net Net-(J1-Pad6): track 0.00 -> 46.1 mm
- net /KP_R3: track 0.00 -> 45.3 mm
- net /KP_C2: track 0.00 -> 39.5 mm
- net Net-(J1-Pad7): track 0.00 -> 35.5 mm
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